File: pcb/e-ink_tap_handle.kicad_sch (KiCad schematic)
At the start: 41 parts, among them IC1 MDBT42Q-512KV2, IC2 LSM6DSLTR, J1 JTAG_SWD_6, J2 USB_C_Receptacle_USB2.0, J3 Conn_01x24, Q1 2N7002E, U1 TP4056, U2 XC6206PxxxMR

Commit message: mall changes to PCB 3v3 routing
Parts:
- added TP (x2): TestPoint, symbol Connector:TestPoint
- U: renamed from J1; value JTAG_SWD_6 -> (none); footprint Connector:Tag-Connect_TC2050-IDC-NL_2x05_P1.27mm_Vertical -> (none)
- U: renamed from R1; value 3k -> (none); footprint Resistor_SMD:R_0603_1608Metric -> (none)
- U: renamed from R2; value 3k -> (none); footprint Resistor_SMD:R_0603_1608Metric -> (none)
- U: renamed from C3; value 10uF -> (none); footprint Capacitor_SMD:C_0603_1608Metric -> (none)
- U: renamed from C1; value 1uF -> (none); footprint Capacitor_SMD:C_0603_1608Metric -> (none)
- U: renamed from C17; value 10uF -> (none); footprint Capacitor_SMD:C_0603_1608Metric -> (none)
- U: renamed from C11; value 1uF -> (none); footprint Capacitor_SMD:C_0603_1608Metric -> (none)
- U: renamed from D4; value RLED -> (none); footprint LED_SMD:LED_0603_1608Metric -> (none)
- U: renamed from C2; value 10uF -> (none); footprint Capacitor_SMD:C_0603_1608Metric -> (none)
- U: renamed from C4; value 4.7uF -> (none); footprint Capacitor_SMD:C_0603_1608Metric -> (none)
- U: renamed from R7; value 2k -> (none); footprint Resistor_SMD:R_0603_1608Metric -> (none)
- U: renamed from C10; value 1uF -> (none); footprint Capacitor_SMD:C_0603_1608Metric -> (none)
- U: renamed from C8; value 1uF -> (none); footprint Capacitor_SMD:C_0603_1608Metric -> (none)
- U: renamed from J3; value Conn_01x24 -> (none); footprint Connector_FFC-FPC:Hirose_FH12-24S-0.5SH_1x24-1MP_P0.50mm_Horizontal -> (none)
- U: renamed from IC1; value MDBT42Q-512KV2 -> (none); footprint MDBT42Q512KV2 -> (none)
- U: renamed from C6; value 1uF -> (none); footprint Capacitor_SMD:C_0603_1608Metric -> (none)
- U: renamed from D2; value MBR0530 -> (none); footprint Diode_SMD:D_SOD-123 -> (none)
- U: renamed from R8; value 806k -> (none); footprint Resistor_SMD:R_0603_1608Metric -> (none)
- U: renamed from U1; value TP4056 -> (none); footprint Package_SO:HSOP-8-1EP_3.9x4.9mm_P1.27mm_EP2.41x3.1mm_ThermalVias -> (none)
- U: renamed from C13; value 1uF -> (none); footprint Capacitor_SMD:C_0603_1608Metric -> (none)
- U: renamed from C14; value 1uF -> (none); footprint Capacitor_SMD:C_0603_1608Metric -> (none)
- U: renamed from U2; value XC6206PxxxMR -> (none); footprint Package_TO_SOT_SMD:SOT-23 -> (none)
- U: renamed from C7; value 10uF -> (none); footprint Capacitor_SMD:C_0603_1608Metric -> (none)
- U: renamed from J2; value USB_C_Receptacle_USB2.0 -> (none); footprint Connector_USB:USB_C_Receptacle_HRO_TYPE-C-31-M-12 -> (none)
- U: renamed from R5; value 5.1k -> (none); footprint Resistor_SMD:R_0603_1608Metric -> (none)
- U: renamed from IC2; value LSM6DSLTR -> (none); footprint Package_LGA:LGA-14_3x2.5mm_P0.5mm_LayoutBorder3x4y -> (none)
- U: renamed from R4; value 5.1k -> (none); footprint Resistor_SMD:R_0603_1608Metric -> (none)
- U: renamed from D5; value MBR0530 -> (none); footprint Diode_SMD:D_SOD-123 -> (none)
- U: renamed from R9; value 2M -> (none); footprint Resistor_SMD:R_0603_1608Metric -> (none)
- U: renamed from L1; value 10uH -> (none); footprint Inductor_SMD:L_0805_2012Metric -> (none)
- U: renamed from Q1; value 2N7002E -> (none); footprint Package_TO_SOT_SMD:SOT-23 -> (none)
- U: renamed from BT1; value 4.2V -> (none); footprint Connector_JST:JST_PH_S2B-PH-SM4-TB_1x02-1MP_P2.00mm_Horizontal -> (none)
- U: renamed from R6; value 2k -> (none); footprint Resistor_SMD:R_0603_1608Metric -> (none)
- U: renamed from R3; value 0.47R -> (none); footprint Resistor_SMD:R_0603_1608Metric -> (none)
- U: renamed from C9; value 1uF -> (none); footprint Capacitor_SMD:C_0603_1608Metric -> (none)
- U: renamed from C5; value 1uF -> (none); footprint Capacitor_SMD:C_0603_1608Metric -> (none)
- U: renamed from D3; value GLED -> (none); footprint LED_SMD:LED_0603_1608Metric -> (none)
- U: renamed from C15; value 1uF -> (none); footprint Capacitor_SMD:C_0603_1608Metric -> (none)
- U: renamed from C16; value 100nf -> (none); footprint Capacitor_SMD:C_0603_1608Metric -> (none)
- U: renamed from C12; value 1uF -> (none); footprint Capacitor_SMD:C_0603_1608Metric -> (none)
- U: renamed from D1; value MBR0530 -> (none); footprint Diode_SMD:D_SOD-123 -> (none)
Connections:
- net GND: now also TP.1
- net at U.1, U.1, U.1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: now also TP.1
